File: hardware/Input.kicad_sch (KiCad schematic)
At the start: 8 parts, among them U5 SFH6206-1T, U6 SFH6206-1T, U7 SFH6206-1T, U8 SFH6206-1T

Commit message: fast fertig
Parts:
- added J1, J2: Conn_01x03, Connector_Phoenix_MKDSx:MKDSN 2,5-2-5.08, symbol Connector_Generic:Conn_01x02
- added R200, R201, R202, R203, R204, R205, R206, R207: R, Resistor_SMD:R_2010_5025Metric_Pad1.40x2.65mm_HandSolder, symbol Device:R
Connections:
- net IN_01: now also R25.2, U8.4; no longer R28.2, U5.4
- net IN_02: now also R26.2, U7.4; no longer R27.2, U6.4
- net IN_03: now also R27.2, U6.4; no longer R26.2, U7.4
- net IN_04: now also R28.2, U5.4; no longer R25.2, U8.4
- net at U6.1: now also R202.2
- net at U6.2: now also R203.2
- net at U5.1: now also R200.2
- net at U5.2: now also R201.2
- net at U8.1: now also R206.2
- net at U8.2: now also R207.2
- net at U7.1: now also R204.2
- net at U7.2: now also R205.2
- new net: J1.2 (Pin_2), R202.1
- new net: J2.1 (Pin_1), R204.1
- new net: J2.2 (Pin_2), R206.1
- new net: J1.1 (Pin_1), R200.1
- new net POWER_N: R201.1, R203.1, R205.1, R207.1
