File: hardware/Relay.kicad_sch (KiCad schematic)
At the start: 32 parts, among them J1 Conn_01x03, J12 Conn_01x03, J13 Conn_01x03, J3 Conn_01x03, J4 Conn_01x03, K1 RT314A12, K2 RT314A12, K3 RT314A12, K4 RT314A12, K5 RT314A12, Q1 BSS123, Q2 BSS123, Q3 BSS123, Q4 BSS123, Q5 BSS123

Commit message: änderung
Parts:
- removed D8: BAS21, Package_TO_SOT_SMD:SOT-23, symbol Diode:BAS21
- removed J13: Conn_01x03, Connector_Phoenix_MC_HighVoltage:PhoenixContact_MCV_1,5_3-G-5.08_1x03_P5.08mm_Vertical, symbol Connector_Generic:Conn_01x03
- removed K5: RT314A12, Relay_THT:Relay_SPDT_Schrack-RT1-16A-FormC_RM5mm, symbol Relay:RT314A12
- removed Q5: BSS123, Package_TO_SOT_SMD:SOT-23, symbol Transistor_FET:BSS123
- removed R22: 100k, Resistor_SMD:R_0603_1608Metric, symbol Device:R
- removed R24: 100, Resistor_SMD:R_0603_1608Metric, symbol Device:R
Connections:
- net K5 is gone; now on net K4: R23.2

Commit message: fast fertig
Parts:
- removed R13: N.P., Resistor_SMD:R_0603_1608Metric, symbol Device:R
- added J5, J6: Conn_01x03, Connector_Phoenix_MKDSx:MKDSN 2,5-2-5.08, symbol Connector_Generic:Conn_01x02
- J1, J3, J4: footprint Connector_Phoenix_MC_HighVoltage:PhoenixContact_MCV_1,5_3-G-5.08_1x03_P5.08mm_Vertical -> Connector_Phoenix_MKDSx:MKDSN 2,5-2-5.08; symbol Connector_Generic:Conn_01x03 -> Connector_Generic:Conn_01x02
- J2: renamed from J12; footprint Connector_Phoenix_MC_HighVoltage:PhoenixContact_MCV_1,5_3-G-5.08_1x03_P5.08mm_Vertical -> Connector_Phoenix_MKDSx:MKDSN 2,5-2-5.08; symbol Connector_Generic:Conn_01x03 -> Connector_Generic:Conn_01x02
Connections:
- net at J2.1 (Pin_1): now also K1.12; no longer K4.12
- net at J2.2 (Pin_2): now also K2.14; no longer K4.11
- net at K4.14: now also J5.1 (Pin_1); no longer J2.3 (Pin_3)
- net at J1.1 (Pin_1): now also K1.14; no longer K1.12
- net at J4.1 (Pin_1): now also K3.11; no longer K2.12
- net at J4.2 (Pin_2): now also K3.14; no longer K2.11
- net at J3.2 (Pin_2): now also K2.12; no longer K3.11
- net at K3.12: now also J5.2 (Pin_2); no longer J3.1 (Pin_1)
- new net: J6.1 (Pin_1), K4.12
- new net: J6.2 (Pin_2), K4.11
- new net: J3.1 (Pin_1), K2.11
