File: hardware/RealyModul_1Wire_ADC.kicad_sch (KiCad schematic)
At the start: 71 parts, among them J1 Conn_01x03, J10 1Wire, J11 1Wire, J2 1Wire, J3 Conn_01x03, J4 Conn_01x03, J5 1Wire, J6 1Wire, J7 1Wire, J8 1Wire, J9 1Wire, K1 RT314A12, K2 RT314A12, K3 RT314A12, Q1 BSS123, Q2 BSS123, Q3 BSS123, U1 LT1129-3.3_SOT223, U2 R-78B5.0-2.0, U3 ESP32-WROOM-32D, U4 ADS1115IDGS

Commit message: Schaltplan angepasst
Parts:
- removed D1, D2, D3: BAS21, Package_TO_SOT_SMD:SOT-23, symbol Diode:BAS21
- removed J1, J3, J4: Conn_01x03, Connector_Phoenix_MC_HighVoltage:PhoenixContact_MCV_1,5_3-G-5.08_1x03_P5.08mm_Vertical, symbol Connector_Generic:Conn_01x03
- removed K1, K2, K3: RT314A12, Relay_THT:Relay_SPDT_Schrack-RT1-16A-FormC_RM5mm, symbol Relay:RT314A12
- removed Q1, Q2, Q3: BSS123, Package_TO_SOT_SMD:SOT-23, symbol Transistor_FET:BSS123
- removed R12, R4, R5: 100k, Resistor_SMD:R_0603_1608Metric, symbol Device:R
- removed R13, R6, R7: 100, Resistor_SMD:R_0603_1608Metric, symbol Device:R
- removed R2: 0R0, Resistor_SMD:R_0603_1608Metric, symbol Device:R
- removed R3: N.P., Resistor_SMD:R_0603_1608Metric, symbol Device:R
Connections:
- net IO33_K3: now also U3.8 (IO32); no longer U3.9 (IO33)
- net IO25_K5: now reaches U3.10 (IO25)
- net INPUT_01: now reaches U3.11 (IO26)
- net INPUT_02: now reaches U3.12 (IO27)
- net INPUT_03: now reaches U3.13 (IO14)
- net INPUT_04: now reaches U3.14 (IO12)
- new net IO32_K4: U3.9 (IO33)
Other:
- added sheet Input (Input.kicad_sch)
- added sheet Relay (Relay.kicad_sch)

Commit message: änderung
Parts:
- removed H1, H2, H3, H4: MOUNT-HOLE3.2, main:3,2, symbol main-eagle-import:MOUNT-HOLE3.2
- removed J6, J7: 1Wire, Connector_JST:JST_XA_B03B-XASK-1-A_1x03_P2.50mm_Vertical, symbol Connector:Screw_Terminal_01x03
- added PS3: IRM-05-5, Converter_ACDC:Converter_ACDC_MeanWell_IRM-05-xx_THT, symbol Converter_ACDC:IRM-05-5
Connections:
- net +5V: now also PS3.4 (+Vo)
- net GND: now also PS3.1 (AC/N), PS3.3 (-Vo)
- net at D6.2 (A), PWR2.1 (Pin_1): now also PS3.2 (AC/L)
- net IO25_K5: no longer names the net of U3.10 (IO25)
Other:
- sheet Relay ports: added none; removed K5

Commit message: fast fertig
Parts:
- removed C5: 100nF/50V, Capacitor_SMD:C_0603_1608Metric, symbol Device:C
- removed D6: ES1D, Diode_SMD:D_SMA, symbol Device:D
- removed J10, J11, J2, J5, J8, J9: 1Wire, Connector_JST:JST_XA_B03B-XASK-1-A_1x03_P2.50mm_Vertical, symbol Connector:Screw_Terminal_01x03
- removed PWR2: Conn_01x02, Connector_Phoenix_MC_HighVoltage:PhoenixContact_MCV_1,5_2-G-5.08_1x02_P5.08mm_Vertical, symbol Connector_Generic:Conn_01x02
- removed U2: R-78B5.0-2.0, Converter_DCDC:Converter_DCDC_RECOM_R-78B-2.0_THT, symbol Regulator_Switching:R-78B5.0-2.0
- added J1: Conn_01x03, Connector_Phoenix_MKDSx:MKDSN 2,5-2-5.08, symbol Connector_Generic:Conn_01x02
- added J10, J8, J9: Conn_01x04, Connector_Phoenix_MC:PhoenixContact_MCV_1,5_4-G-3.81_1x04_P3.81mm_Vertical, symbol Connector_Generic:Conn_01x04
Connections:
- net +3.3V: now also J10.1 (Pin_1), J8.1 (Pin_1), J9.1 (Pin_1)
- net 1Wire: now also J10.3 (Pin_3), J10.4 (Pin_4)
- net GND: now also J10.2 (Pin_2), J8.2 (Pin_2), J9.2 (Pin_2); no longer PS3.1 (AC/N)
- net at PS3.2 (AC/L): now also J1.1 (Pin_1)
- net at R16.1: now also J9.3 (Pin_3)
- net at R17.1: now also J9.4 (Pin_4)
- net at R15.1: now also J8.4 (Pin_4)
- net at R14.1: now also J8.3 (Pin_3)
- new net POWER_N: J1.2 (Pin_2), PS3.1 (AC/N)
Other:
- sheet Input ports: added POWER_N; removed none
- moved on the sheet: PS3, R1

Commit message: fertig
Parts:
- removed FLASH1, RES1: SPST_TACT-EVQQ2, main:EVQ-Q2, symbol main-eagle-import:SPST_TACT-EVQQ2
- removed J8, J9: Conn_01x04, Connector_Phoenix_MC:PhoenixContact_MCV_1,5_4-G-3.81_1x04_P3.81mm_Vertical, symbol Connector_Generic:Conn_01x04
- removed PS3: IRM-05-5, Converter_ACDC:Converter_ACDC_MeanWell_IRM-05-xx_THT, symbol Converter_ACDC:IRM-05-5
- added J11, J13, J8, J9: Conn_01x02, Connector_Phoenix_MKDSx:MKDS_1_2_3.81, symbol Connector_Generic:Conn_01x02
- added PS1: IRM-05-5, Converter_ACDC:Converter_ACDC_MeanWell_IRM-05-xx_THT, symbol Converter_ACDC:IRM-05-5
- J10: value Conn_01x04 -> Conn_01x03; footprint Connector_Phoenix_MC:PhoenixContact_MCV_1,5_4-G-3.81_1x04_P3.81mm_Vertical -> Connector_Phoenix_MKDSx:MKDS_1_3_3.81; symbol Connector_Generic:Conn_01x04 -> Connector_Generic:Conn_01x03
- R1: value 4K7 -> 4k7
Connections:
- net +3.3V: now also R1.1, J11.2 (Pin_2), J8.2 (Pin_2); no longer R1.2
- net +5V: now also PS1.4 (+Vo)
- net 1Wire: now also R1.2; no longer J10.4 (Pin_4), R1.1
- net GND: now also J11.1 (Pin_1), J8.1 (Pin_1), PS1.3 (-Vo)
- net POWER_N: now also PS1.1 (AC/N)
- net at J1.1 (Pin_1): now also PS1.2 (AC/L)
- net at R14.1: now also J9.2 (Pin_2)
- net at R15.1: now also J9.1 (Pin_1)
- net at R16.1: now also J13.2 (Pin_2)
- net at R17.1: now also J13.1 (Pin_1)
